Commit message: imu_testing

File: minesweeper_description/urdf/minesweeper.urdf.xacro (robot description, xacro)
@@ -24,4 +24,12 @@
       </collision>
     </link>
+    <link name="imu_link"/>
+    <joint name="imu_joint" type="fixed">
+      <origin xyz="0.375 0.0 0.075" rpy="0.0 0.0 0.0"/>
+      <parent link="base_link"/>
+      <child link="imu_link"/>
+    </joint>
+    <gazebo reference="imu_link">
+    </gazebo>
     <link name="base_footprint"/>
     <joint name="base_footprint_joint" type="fixed">

Commit message: Fixed URDF, Gazebo and Kalman config

File: minesweeper_description/urdf/minesweeper.urdf.xacro (robot description, xacro)
@@ -55,3 +55,17 @@
       </plugin>
     </gazebo>
+    <!--<gazebo>
+      <plugin name="imu_controller" filename="libhector_gazebo_ros_imu.so">
+        <robotNamespace>$(arg robot_namespace)</robotNamespace>
+        <updateRate>50.0</updateRate>
+        <bodyName>base_link</bodyName>
+        <topicName>imu/data</topicName>
+        <accelDrift>0.005 0.005 0.005</accelDrift>
+        <accelGaussianNoise>0.005 0.005 0.005</accelGaussianNoise>
+        <rateDrift>0.005 0.005 0.005 </rateDrift>
+        <rateGaussianNoise>0.005 0.005 0.005 </rateGaussianNoise>
+        <headingDrift>0.005</headingDrift>
+        <headingGaussianNoise>0.005</headingGaussianNoise>
+      </plugin>
+    </gazebo>-->
 </robot>

File: minesweeper_description/urdf/wheel.urdf.xacro (robot description, xacro)
@@ -21,10 +21,10 @@
             <!--<origin xyz="0.17982 0.32146 0.02496" rpy="0 0 0"/>-->
             <mass value="3.1041" />
-            <inertia ixx="9.0731E-05" ixy="4.2946E-13" ixz="-6.6251E-14" iyy="2.038E-07" iyz="1.3211E-06" izz="9.0527E-05"/>
+            <inertia  ixx="0.02467" ixy="0" ixz="0" iyy="0.04411" iyz="0" izz="0.02467" />
           </inertial>
       </link>
       <gazebo reference="${prefix}_wheel_link">
-  			<mu1 value="400.0"/>
-  			<mu2 value="100.0"/>
+  			<mu1 value="1.0"/>
+  			<mu2 value="1.0"/>
   			<kp value="10000000.0" />
   			<kd value="1.0" />

Commit message: Updated URDF and a new RViz package

File: minesweeper_description/urdf/minesweeper.urdf.xacro (robot description, xacro)
@@ -1,10 +1,10 @@
 <?xml version="1.0"?>
-<robot name="wheel" xmlns:xacro="https://github.com/zoidberg2010eaf/minesweeper">
+<robot name="minesweeper" xmlns:xacro="http://www.ros.org/wiki/xacro">
     <xacro:arg name="robot_namespace" default="/" />
     <xacro:include filename="$(find minesweeper_description)/urdf/wheel.urdf.xacro"/>
     <link name="base_link">
       <inertial>
-        <origin xyz="0.0 0.0 0.05045" rpy="0 0 0" />
-        <mass value="23.176" />
+        <origin xyz="0.0 0.0 -0.07796" rpy="0.0 0.0 0.0"/>
+        <mass value="20.25"/>
         <inertia ixx="0.6022" ixy="-0.02364" ixz="-0.1197" iyy="1.7386" iyz="-0.001544" izz="2.0296" />
       </inertial>
@@ -13,15 +13,24 @@
           <mesh filename="package://minesweeper_description/meshes/base_link.STL" />
         </geometry>
-        <material name="yellow">
-          <color rgba="1.0 0.8 0.0 1" />
+        <material name="beige">
+          <color rgba="0.91 0.815 0.592 1" />
         </material>
       </visual>
       <collision>
         <geometry>
-          <box size="0.75 0.50 0.15"/>
+          <box size=".77689 0.422 0.15592"/>
         </geometry>
-        <origin xyz="0.0 0.0 0.075"/>
+        <origin xyz="0.0 0.0 0.07796"/>
       </collision>
     </link>
+    <gazebo reference="base_link">
+      <visual name="base_link_visual">
+          <material>
+              <diffuse>0.91 0.815 0.592 1.0</diffuse>
+              <specular>0.91 0.815 0.592 1.0</specular>
+              <ambient>0.91 0.815 0.592 1.0</ambient>
+          </material>
+      </visual>
+    </gazebo>
     <link name="imu_link"/>
     <joint name="imu_joint" type="fixed">
@@ -38,15 +47,35 @@
       <child link="base_footprint" />
     </joint>
+    <link name="coil_link">
+        <visual>
+            <geometry>
+                <mesh filename="package://minesweeper_description/meshes/coil.dae"/>
+            </geometry>
+        </visual>
+    </link>
+    <joint name="coil" type="fixed">
+        <parent link="base_link"/>
+        <child link="coil_link"/>
+        <origin xyz="0.355 0.0 0.022"/>
+    </joint>
+    <gazebo reference="coil_link">
+      <visual name="base_link_visual">
+          <material>
+            <script>Gazebo/WoodPallet</script>
+            <ambient>0.25 0.25 0.25 1.0</ambient>
+          </material>
+      </visual>
+    </gazebo>
     <xacro:wheel prefix="front_left" angle="0.0">
-      <origin xyz="0.181 0.320 0.025"/>
+      <origin xyz="0.16807 0.161 0.05268"/>
     </xacro:wheel>
     <xacro:wheel prefix="front_right" angle="180.0">
-      <origin xyz="0.181 -0.320 0.025"/>
+      <origin xyz="0.16907 -0.161 0.05268"/>
     </xacro:wheel>
     <xacro:wheel prefix="rear_left" angle="0.0">
-      <origin xyz="-0.181 0.320 0.025"/>
+      <origin xyz="-0.18733 0.161 0.05268"/>
     </xacro:wheel>
     <xacro:wheel prefix="rear_right" angle="180.0">
-      <origin xyz="-0.181 -0.320 0.025"/>
+      <origin xyz="-0.18633 -0.161 0.05268"/>
     </xacro:wheel>
     <gazebo>
@@ -55,5 +84,5 @@
       </plugin>
     </gazebo>
-    <!--<gazebo>
+    <gazebo>
       <plugin name="imu_controller" filename="libhector_gazebo_ros_imu.so">
         <robotNamespace>$(arg robot_namespace)</robotNamespace>
@@ -68,4 +97,4 @@
         <headingGaussianNoise>0.005</headingGaussianNoise>
       </plugin>
-    </gazebo>-->
+    </gazebo>
 </robot>

File: minesweeper_description/urdf/wheel.urdf.xacro (robot description, xacro)
@@ -1,4 +1,4 @@
 <?xml version="1.0"?>
-<robot name="wheel" xmlns:xacro="https://github.com/zoidberg2010eaf/minesweeper">
+<robot name="wheel" xmlns:xacro="http://www.ros.org/wiki/xacro">
     <xacro:macro name="wheel" params="prefix angle *joint_origin">
       <link name="${prefix}_wheel_link">
@@ -14,14 +14,22 @@
           <collision>
               <geometry>
-                  <cylinder radius="0.165" length="0.11"/>
+                  <cylinder radius="0.15955" length="0.100"/>
               </geometry>
-              <origin xyz="0.0 0.0 0.0" rpy="0 ${radians(90)} ${radians(90)}"/>
+              <origin xyz="0.0 ${0.125*cos(radians(angle))} 0.0" rpy="0 ${radians(90)} ${radians(90)}"/>
           </collision>
           <inertial>
-            <!--<origin xyz="0.17982 0.32146 0.02496" rpy="0 0 0"/>-->
-            <mass value="3.1041" />
+            <mass value="2.8" />
             <inertia  ixx="0.02467" ixy="0" ixz="0" iyy="0.04411" iyz="0" izz="0.02467" />
           </inertial>
       </link>
+      <gazebo reference="${prefix}_wheel_link">
+        <visual name="{prefix}_wheel_visual">
+            <material>
+                <diffuse>0.05 0.05 0.05 1.0</diffuse>
+                <specular>0.05 0.05 0.05 1.0</specular>
+                <ambient>0.05 0.05 0.05 1.0</ambient>
+            </material>
+        </visual>
+      </gazebo>
       <gazebo reference="${prefix}_wheel_link">
   			<mu1 value="1.0"/>

Commit message: Tweaks for mapping

File: minesweeper_description/urdf/minesweeper.urdf.xacro (robot description, xacro)
@@ -57,6 +57,6 @@
         <parent link="base_link"/>
         <child link="coil_link"/>
-        <origin xyz="0.355 0.0 0.022"/>
-    </joint>
+        <origin xyz="0.355 0.0 0.04"/>
+    </joint>pose
     <gazebo reference="coil_link">
       <visual name="base_link_visual">
@@ -67,4 +67,11 @@
       </visual>
     </gazebo>
+    <link name="coil_center_link">
+    </link>
+    <joint name="coil_center" type="fixed">
+        <parent link="coil_link"/>
+        <child link="coil_center_link"/>
+        <origin xyz="0.190 0.0 -0.1"/>
+    </joint>
     <xacro:wheel prefix="front_left" angle="0.0">
       <origin xyz="0.16807 0.161 0.05268"/>

Commit message: day 3 of testing and tweaking

File: minesweeper_description/urdf/minesweeper.urdf.xacro (robot description, xacro)
@@ -35,5 +35,5 @@
     <link name="imu_link"/>
     <joint name="imu_joint" type="fixed">
-      <origin xyz="0.375 0.0 0.075" rpy="0.0 0.0 0.0"/>
+      <origin xyz="0.0 0.0 0.075" rpy="0.0 0.0 0.0"/>
       <parent link="base_link"/>
       <child link="imu_link"/>
@@ -91,5 +91,5 @@
       </plugin>
     </gazebo>
-    <gazebo>
+    <!--<gazebo>
       <plugin name="imu_controller" filename="libhector_gazebo_ros_imu.so">
         <robotNamespace>$(arg robot_namespace)</robotNamespace>
@@ -104,4 +104,4 @@
         <headingGaussianNoise>0.005</headingGaussianNoise>
       </plugin>
-    </gazebo>
+    </gazebo>-->
 </robot>

Commit message: rqt map is almost done

File: minesweeper_description/urdf/minesweeper.urdf.xacro (robot description, xacro)
@@ -72,5 +72,5 @@
         <parent link="coil_link"/>
         <child link="coil_center_link"/>
-        <origin xyz="0.190 0.0 -0.1"/>
+        <origin xyz="0.290 0.0 -0.1"/> <!--it was 0.190 in the x-->
     </joint>
     <xacro:wheel prefix="front_left" angle="0.0">

Commit message: Updated the URDF

File: minesweeper_description/urdf/minesweeper.urdf.xacro (robot description, xacro)
@@ -2,5 +2,5 @@
 <robot name="minesweeper" xmlns:xacro="http://www.ros.org/wiki/xacro">
     <xacro:arg name="robot_namespace" default="/" />
-    <xacro:include filename="$(find minesweeper_description)/urdf/wheel.urdf.xacro"/>
+    <xacro:include filename="$(find shit)/urdf/wheel.urdf.xacro"/>
     <link name="base_link">
       <inertial>
@@ -75,14 +75,14 @@
     </joint>
     <xacro:wheel prefix="front_left" angle="0.0">
-      <origin xyz="0.16807 0.161 0.05268"/>
+      <origin xyz="0.15 0.2105 0.03118"/>
     </xacro:wheel>
     <xacro:wheel prefix="front_right" angle="180.0">
-      <origin xyz="0.16907 -0.161 0.05268"/>
+      <origin xyz="0.15 -0.2105 0.03118"/>
     </xacro:wheel>
     <xacro:wheel prefix="rear_left" angle="0.0">
-      <origin xyz="-0.18733 0.161 0.05268"/>
+      <origin xyz="-0.205 0.2105 0.03118"/>
     </xacro:wheel>
     <xacro:wheel prefix="rear_right" angle="180.0">
-      <origin xyz="-0.18633 -0.161 0.05268"/>
+      <origin xyz="-0.205 -0.2105 0.03118"/>
     </xacro:wheel>
     <gazebo>
@@ -91,5 +91,5 @@
       </plugin>
     </gazebo>
-    <!--<gazebo>
+    <gazebo>
       <plugin name="imu_controller" filename="libhector_gazebo_ros_imu.so">
         <robotNamespace>$(arg robot_namespace)</robotNamespace>
@@ -104,4 +104,4 @@
         <headingGaussianNoise>0.001</headingGaussianNoise>
       </plugin>
-    </gazebo>-->
+    </gazebo>
 </robot>

Commit message: FML

File: minesweeper_description/urdf/minesweeper.urdf.xacro (robot description, xacro)
@@ -35,5 +35,5 @@
     <link name="imu_link"/>
     <joint name="imu_joint" type="fixed">
-      <origin xyz="0.0 0.0 0.075" rpy="0.0 0.0 0.0"/>
+      <origin xyz="-0.05 0.0 0.03118" rpy="0.0 0.0 0.0"/>
       <parent link="base_link"/>
       <child link="imu_link"/>
@@ -50,6 +50,9 @@
         <visual>
             <geometry>
-                <mesh filename="package://minesweeper_description/meshes/coil.dae"/>
+                <mesh filename="package://minesweeper_description/meshes/coil_link.STL"/>
             </geometry>
+            <material name="gray">
+              <color rgba="0.8 0.8 0.8 1" />
+            </material>
         </visual>
     </link>
@@ -57,14 +60,6 @@
         <parent link="base_link"/>
         <child link="coil_link"/>
-        <origin xyz="0.355 0.0 0.04"/>
-    </joint>pose
-    <gazebo reference="coil_link">
-      <visual name="base_link_visual">
-          <material>
-            <script>Gazebo/WoodPallet</script>
-            <ambient>0.25 0.25 0.25 1.0</ambient>
-          </material>
-      </visual>
-    </gazebo>
+        <origin xyz="0.2165 0.0 0.04" rpy="0.0 0.0 -1.57079"/>
+    </joint>
     <link name="coil_center_link">
     </link>
@@ -72,5 +67,5 @@
         <parent link="coil_link"/>
         <child link="coil_center_link"/>
-        <origin xyz="0.290 0.0 -0.1"/> <!--it was 0.190 in the x-->
+        <origin xyz="0.0 0.307 -0.1"/> <!--it was 0.190 in the x-->
     </joint>
     <xacro:wheel prefix="front_left" angle="0.0">
@@ -97,9 +92,9 @@
         <bodyName>imu_link</bodyName>
         <topicName>imu/data</topicName>
-        <accelDrift>0.001 0.001 0.001</accelDrift>
-        <accelGaussianNoise>0.001 0.001 0.001</accelGaussianNoise>
-        <rateDrift>0.001 0.001 0.001</rateDrift>
-        <rateGaussianNoise>0.001 0.001 0.001</rateGaussianNoise>
-        <headingDrift>0.001</headingDrift>
+        <accelDrift>0.005 0.005 0.005</accelDrift>
+        <accelGaussianNoise>0.005 0.005 0.005</accelGaussianNoise>
+        <rateDrift>0.005 0.005 0.005</rateDrift>
+        <rateGaussianNoise>0.005 0.005 0.005</rateGaussianNoise>
+        <headingDrift>0.005</headingDrift>
         <headingGaussianNoise>0.001</headingGaussianNoise>
       </plugin>
